File: EfficientInterface/EfficientInterface.kicad_pcb (KiCad board)
At the start: 4 copper layers, 58.4 x 41.9 mm, 41 parts, among them J1 DF40HC(3.0)-70DS-0.4V(51), J2 DF40HC(3.0)-70DS-0.4V(51), J3 SFH11-PBPC-D05-ST-BK, J4 SFH11-PBPC-D05-ST-BK, J5 SFH11-PBPC-D05-ST-BK, J6 SFH11-PBPC-D05-ST-BK

Commit message: Updated Files
Other:
- board text added: "Efficient E1x Stamp Interface Carnegie Mellon University Made by Neil Khera v1.0"
- board text removed: "Efficient E1x Stamp Interface Carnegie Mellon University v1.0"
Changed lines of the file:
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@@
 		)
 	)
-	(gr_text "Efficient E1x Stamp Interface\nCarnegie Mellon University\nv1.0"
+	(gr_text "Efficient E1x Stamp Interface\nCarnegie Mellon University\nMade by Neil Khera\nv1.0"
 		(at 155.575 114.173 0)
 		(layer "B.SilkS")
