File: EfficientStamp/EfficientStamp.kicad_pcb (KiCad board)
At the start: 6 copper layers, 38.1 x 38.1 mm, 103 parts, among them J1 TC2050, J2 TC2050, J3 DF40C-70DP-0.4V(51), J4 DF40C-70DP-0.4V(51), SW1 B3U-1000P, U1 Efficient E1x, U2 MSP430F5151IRSBT, U3 TPS22916BYFPR, U4 IS25WJ032F-JNLE, Y1 ECS-2520MVLC-500-CN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

Commit message: Updated Files
Other:
- board text added: "Made by Neil Khera"
Changed lines of the file:
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@@
+		)
+	)
+	(gr_text "Made by Neil Khera"
+		(at 120.33 113.5888 0)
+		(layer "B.SilkS")
+		(effects
+			(font
+				(size 0.635 0.635)
+				(thickness 0.127)
+				(bold yes)
+			)
+			(justify mirror)
 		)
 	)
